Commit message: Fixed colours

File: description/robot_core.xacro (robot description, xacro)
@@ -3,5 +3,5 @@
      <xacro:include filename="inertial_macros.xacro"/>
     <material name="white">
-        <color rgba="1 1 1 1"/>
+        <color rgba="1 1 1 1" />
     </material>
     <material name="orange">
@@ -29,5 +29,5 @@
                 <box size="0.35 0.35 0.15" />
             </geometry>
-            <material name="white" />
+            <material name="white"/>
         </visual>
         <collision>
@@ -52,6 +52,6 @@
             <geometry>
                 <cylinder radius="0.05" length="0.04" />
-                <material name="blue" />
             </geometry>
+             <material name="blue"/>
         </visual>
         <collision>
@@ -75,6 +75,6 @@
             <geometry>
                 <cylinder radius="0.05" length="0.04" />
-                <material name="blue" />
             </geometry>
+             <material name="blue"/>
         </visual>
         <collision>
@@ -97,6 +97,6 @@
             <geometry>
                 <sphere radius="0.05" />
-                <material name="black" />
             </geometry>
+            <material name="black"/>
         </visual>
         <collision>

Commit message: Added Lidar

File: description/robot_core.xacro (robot description, xacro)
@@ -13,4 +13,7 @@
     <material name="black">
         <color rgba="0 0 0 1"/>
+    </material>
+     <material name="red">
+        <color rgba="1 0 0 1"/>
     </material>
     <!-- BASE Link -->

Commit message: Updated wheel size, separation and encoder values

File: description/robot_core.xacro (robot description, xacro)
@@ -6,5 +6,5 @@
     <xacro:property name="chassis_height" value="0.10"/>
     <xacro:property name="chassis_mass" value="1.0"/>
-    <xacro:property name="wheel_radius" value="0.034"/>
+    <xacro:property name="wheel_radius" value="0.033"/>
     <xacro:property name="wheel_thickness" value="0.026"/>
     <xacro:property name="wheel_mass" value="0.05"/>

File: description/ros2_control.xacro (robot description, xacro)
@@ -11,5 +11,5 @@
                 <param name="baud_rate">57600</param>
                 <param name="timeout_ms">1000</param>
-                <param name="enc_counts_per_rev">3436</param>
+                <param name="enc_counts_per_rev">1950</param>
             </hardware>
             <joint name="left_wheel_joint">

Commit message: Added IMU to descr

File: description/robot_core.xacro (robot description, xacro)
@@ -67,4 +67,26 @@
     </link>
     <gazebo reference="chassis">
+        <material>Gazebo/Orange</material>
+    </gazebo>
+     <!-- IMU Link -->
+    <link name="imu_link">
+    <visual>
+        <origin xyz="0 0 0" rpy="0 0 0"/>
+        <geometry>
+            <box size="0.01 0.01 0.01"/>  <!-- tiny box for IMU -->
+        </geometry>
+        <material name="Grey">
+            <color rgba="0.5 0.5 0.5 1.0"/>
+        </material>
+    </visual>
+    </link>
+    <!-- Static Joint Between Base and IMU -->
+    <joint name="imu_joint" type="fixed">
+        <parent link="base_link"/>
+        <child link="imu_link"/>
+        <!-- Replace xyz and rpy with actual physical mounting position -->
+        <origin xyz="0.0 0.0 0.05" rpy="0 0 0"/>
+    </joint>
+     <gazebo reference="imu_link">
         <material>Gazebo/Orange</material>
     </gazebo>
